Commit message: removed max contacts tag, urdf file and changed display.launch to just load the xacro
also added friction and damping to joints and changed center of mass

File: Wheelchair 1.0/wheelchair_1_description/urdf/wheelchair.urdf.xacro (robot description, xacro)
@@ -6,5 +6,5 @@
   	<link name='base_link'>
 	    <visual>
-	    	<oririn rpy= "0 -0 0" xyx = "-0.24919 -1.2e-05 -0.357491"/>
+	    	<origin rpy= "0 -0 0" xyz = "0 0 0"/>
 		    <geometry>
 		    	<mesh scale=" 1 1 1" filename = "package://wheelchair_1_description/meshes/Wheelchair-base_col.STL"/>
@@ -12,5 +12,5 @@
 	    </visual>
 	    <collision>
-        	<oririn rpy= "0 -0 0" xyx = "-0.24919 -1.2e-05 -0.357491"/>
+        	<origin rpy= "0 -0 0" xyz = "0 0 0"/>
         	<geometry>
           		<mesh scale=" 1 1 1" filename = "package://wheelchair_1_description/meshes/Wheelchair-base_col.STL"/>
@@ -18,4 +18,5 @@
       	</collision>
 	    <inertial>
+			<origin rpy= "0 -0 0" xyz = "0.2 0 0"/>
         	<mass value="54.78178"/>
          	<inertia ixx="0.253724" ixy="7e-06" ixz="0.022948" iyy="0.218409" iyz="7e-06" izz="0.382313"/>
@@ -54,5 +55,5 @@
       	</collision>
 		<inertial>
-        	<mass value="0.279084"/>
+        	<mass value="0.279085"/>
          	<inertia ixx="0.000442" ixy="1e-06" ixz="0.000123" iyy="0.000458" iyz="8e-06" izz="0.000182"/>
  	    </inertial>
@@ -72,11 +73,11 @@
       	</collision>
 	  	<inertial>
-        	<mass value="2.91669"/>
-         	<inertia ixx="0.112302" ixy="0" ixz="0.0" iyy="0.222779" iyz="0.0" izz="0.112302"/>
+        	<mass value="4.08233"/>
+         	<inertia ixx="0.112302" ixy="0" ixz="0" iyy="0.222779" iyz="0" izz="0.112302"/>
  	    </inertial>
   	</link>
   	<link name="Right-Caster-Wheel">
 	  	<visual>
-	  		<origin rpy = "0 -0 0" xyz = "-0.32661 0.24108 -0.06"/>
+	  		<origin rpy = "0 -0 0" xyz = "-0.32661 0.24669 -0.06"/>
 	  		<geometry>
 	  			<mesh scale=" 1 1 1" filename = "package://wheelchair_1_description/meshes/Right-Caster-Wheel.STL"/>
@@ -84,5 +85,5 @@
 	  	</visual>
 	  	<collision>
-        	<origin rpy  = "0 -0 0" xyz = "-0.32661 0.24108 -0.06"/>
+        	<origin rpy  = "0 -0 0" xyz = "-0.32661 0.24669 -0.06"/>
         	<geometry>
           		<mesh scale=" 1 1 1" filename = "package://wheelchair_1_description/meshes/Right-Caster-Wheel_col.STL"/>
@@ -126,5 +127,5 @@
       	</collision>
 	  	<inertial>
-	        <mass value="2.91699"/>
+	        <mass value="4.08233"/>
 	        <inertia ixx="0.112302" ixy="0" ixz="0" iyy="0.222779" iyz="0" izz="0.112302"/>
  	    </inertial>
@@ -135,5 +136,6 @@
 	   <origin xyz="-0.04295 -0.00183 -0.0917"/>
 	   <axis xyz="0 1 0"/>
-	   <limit effort= "100" lower = "${lower}" upper = "${upper}" velocity = "10"/>
+	   <limit effort= "10" lower = "${lower}" upper = "${upper}" velocity = "10"/>
+	   <dynamics damping = ".7" friction ="1.5"/>
 	</joint>
 	<joint name="Wheelchair-base-Left-Caster-Yaw" type="revolute">
@@ -143,4 +145,5 @@
 	   <axis xyz="0 0 -1"/>
 	   <limit effort= "100" lower = "${lower}" upper = "${upper}" velocity = "10"/>
+	   <dynamics damping = "0.7" friction ="1.5"/>
 	</joint>
 	<joint name="Wheelchair_base_Left_Wheel" type="revolute">
@@ -150,4 +153,5 @@
 	   <axis xyz="0 1 0"/>
 	   <limit effort= "100" lower = "${lower}" upper = "${upper}" velocity = "10"/>
+	   <dynamics damping = "0" friction ="0"/>
 	</joint>
 	<joint name="Right-Caster-Yaw-Right-Caster-Wheel" type="revolute">
@@ -164,4 +168,5 @@
 	   <axis xyz="0 0 1"/>
 	   <limit effort= "100" lower = "${lower}" upper = "${upper}" velocity = "10"/>
+	   <dynamics damping = "0.7" friction ="1.5"/>
 	</joint>
 	<joint name="Wheelchair_base_Right_Wheel" type="revolute">
@@ -171,4 +176,5 @@
 	   <axis xyz="0 1 0"/>
 	   <limit effort= "100" lower = "${lower}" upper = "${upper}" velocity = "10"/>
+	   <dynamics damping = "0" friction ="0"/>
 	</joint>
     <transmission name="Wheelchair_base_Left_Wheel-trans">
