Commit message: fixed recording, merge files

File: Wheelchair_1/wheelchair_description_1/Archive/wheelchair.urdf.xacro (robot description, xacro)
@@ -18,5 +18,5 @@
       	</collision>
 	    <inertial>
-        	<mass value="54.78178"/>
+        	<mass value="4.78178"/>
          	<inertia ixx="0.253724" ixy="7e-06" ixz="0.022948" iyy="0.218409" iyz="7e-06" izz="0.382313"/>
  	    </inertial>
@@ -144,5 +144,5 @@
 	   <limit effort= "100" lower = "${lower}" upper = "${upper}" velocity = "10"/>
 	</joint>
-	<joint name="Wheelchair_base_Left_Wheel" type="revolute">
+	<joint name="Wheelchair-base-Left-Wheel" type="revolute">
 	   <parent link="base_link"/>
 	   <child link="Left-Wheel"/>
@@ -165,5 +165,5 @@
 	   <limit effort= "100" lower = "${lower}" upper = "${upper}" velocity = "10"/>
 	</joint>
-	<joint name="Wheelchair_base_Right_Wheel" type="revolute">
+	<joint name="Wheelchair-base-Right-Wheel" type="revolute">
 	   <parent link="base_link"/>
 	   <child link="Right-Wheel"/>
@@ -172,22 +172,20 @@
 	   <limit effort= "100" lower = "${lower}" upper = "${upper}" velocity = "10"/>
 	</joint>
-    <transmission name="Wheelchair_base_Left_Wheel-trans">
+    <transmission name="Wheelchair-base-Left-Wheel-trans">
       	<type>transmission_interface/SimpleTransmission</type>
-      	<actuator name="Wheelchair_base_Left_Wheel-motor">
+      	<actuator name="Wheelchair-base-Left-Wheel-motor">
         	<mechanicalReduction>1</mechanicalReduction>
      	</actuator>
-      	<joint name="Wheelchair_base_Left_Wheel">
-        	<hardwareInterface>hardware_interface/VelocityJointInterface</hardwareInterface>
-        	<!-- <hardwareInterface>hardware_interface/EffortJointInterface</hardwareInterface> -->
+      	<joint name="Wheelchair-base-Left-Wheel">
+        	<hardwareInterface>VelocityJointInterface</hardwareInterface>
       	</joint>
     </transmission>
-    <transmission name="Wheelchair_base_Right_Wheel-trans">
+    <transmission name="Wheelchair-base-Right-Wheel-trans">
       	<type>transmission_interface/SimpleTransmission</type>
-      	<actuator name="Wheelchair_base_Right_Wheel-motor">
+      	<actuator name="Wheelchair-base-Right-Wheel-motor">
         	<mechanicalReduction>1</mechanicalReduction>
       	</actuator>
-      	<joint name="Wheelchair_base_Right_Wheel">
-        	<hardwareInterface>hardware_interface/VelocityJointInterface</hardwareInterface>
-        	<!-- <hardwareInterface>hardware_interface/EffortJointInterface</hardwareInterface> -->
+      	<joint name="Wheelchair-base-Right-Wheel">
+        	<hardwareInterface>VelocityJointInterface</hardwareInterface>
       	</joint>
     </transmission>

File: Wheelchair_1/wheelchair_description_1/Archive/wheelchairvelcon.urdf.xacro (robot description, xacro)
@@ -1,5 +1,5 @@
 <?xml version="1.0" encoding="utf-8"?>
 <robot name="wheelchair" xmlns:xacro="http://www.ros.org/wiki/xacro">
-	<xacro:include filename="$(find wheelchair_description_1)/urdf/wheelchair.gazebo" />
+	<xacro:include filename="$(find wheelchair_1_description)/urdf/wheelchair.gazebo"/>
 	<xacro:property name = "lower" value = "-1000"/>
 	<xacro:property name = "upper" value = "1000"/>
@@ -8,5 +8,5 @@
 	    	<oririn rpy= "0 -0 0" xyx = "-0.24919 -1.2e-05 -0.357491"/>
 		    <geometry>
-		    	<mesh scale=" 1 1 1" filename = "package://wheelchair_description_1/meshes/Wheelchair-base_col.STL"/>
+		    	<mesh scale=" 1 1 1" filename = "package://wheelchair_1_description/meshes/Wheelchair-base_col.STL"/>
 		    </geometry>
 	    </visual>
@@ -14,5 +14,5 @@
         	<oririn rpy= "0 -0 0" xyx = "-0.24919 -1.2e-05 -0.357491"/>
         	<geometry>
-          		<mesh scale=" 1 1 1" filename = "package://wheelchair_description_1/meshes/Wheelchair-base_col.STL"/>
+          		<mesh scale=" 1 1 1" filename = "package://wheelchair_1_description/meshes/Wheelchair-base_col.STL"/>
         	</geometry>
       	</collision>
@@ -26,5 +26,5 @@
 	  		<origin rpy = "0 -0 0" xyz = "-0.32661 -0.24669 -0.06"/>
 	  		<geometry>
-	  			<mesh scale=" 1 1 1" filename = "package://wheelchair_description_1/meshes/Left-Caster-Wheel.STL"/>
+	  			<mesh scale=" 1 1 1" filename = "package://wheelchair_1_description/meshes/Left-Caster-Wheel.STL"/>
 	  		</geometry>
 	  	</visual>
@@ -32,5 +32,5 @@
         	<origin rpy = "0 -0 0" xyz = "-0.32661 -0.24669 -0.06"/>
         		<geometry>
-          			<mesh scale=" 1 1 1" filename = "package://wheelchair_description_1/meshes/Left-Caster-Wheel_col.STL"/>
+          			<mesh scale=" 1 1 1" filename = "package://wheelchair_1_description/meshes/Left-Caster-Wheel_col.STL"/>
         		</geometry>
      	</collision>
@@ -44,5 +44,5 @@
 		  	<origin rpy = "0 -0 0"  xyz = "-0.35956 -0.24291 -0.1517"/>
 		  	<geometry>
-		  		<mesh scale=" 1 1 1" filename = "package://wheelchair_description_1/meshes/Left-Caster-Yaw.STL"/>
+		  		<mesh scale=" 1 1 1" filename = "package://wheelchair_1_description/meshes/Left-Caster-Yaw.STL"/>
 		  	</geometry>
 		</visual>
@@ -50,5 +50,5 @@
           	<origin rpy = "0 -0 0" xyz = "-0.35956 -0.24291 -0.1517"/>
           	<geometry>
-            	<mesh scale=" 1 1 1" filename = "package://wheelchair_description_1/meshes/Left-Caster-Yaw_col.STL"/>
+            	<mesh scale=" 1 1 1" filename = "package://wheelchair_1_description/meshes/Left-Caster-Yaw_col.STL"/>
           	</geometry>
       	</collision>
@@ -62,5 +62,5 @@
 	  		<origin rpy  = "0 -0 0" xyz = "-0 -0.26808 -0.305"/>
 	  		<geometry>
-		  		<mesh scale=" 1 1 1" filename = "package://wheelchair_description_1/meshes/Left-Wheel.STL"/>
+		  		<mesh scale=" 1 1 1" filename = "package://wheelchair_1_description/meshes/Left-Wheel.STL"/>
 		  	</geometry>
 	  	</visual>
@@ -68,5 +68,5 @@
         	<origin rpy  = "0 -0 0" xyz = "-0 -0.26808 -0.305"/>
         	<geometry>
-          		<mesh scale=" 1 1 1" filename = "package://wheelchair_description_1/meshes/Left-Wheel_col.STL"/>
+          		<mesh scale=" 1 1 1" filename = "package://wheelchair_1_description/meshes/Left-Wheel_col.STL"/>
         	</geometry>
       	</collision>
@@ -80,5 +80,5 @@
 	  		<origin rpy = "0 -0 0" xyz = "-0.32661 0.24108 -0.06"/>
 	  		<geometry>
-	  			<mesh scale=" 1 1 1" filename = "package://wheelchair_description_1/meshes/Right-Caster-Wheel.STL"/>
+	  			<mesh scale=" 1 1 1" filename = "package://wheelchair_1_description/meshes/Right-Caster-Wheel.STL"/>
 	  		</geometry>
 	  	</visual>
@@ -86,5 +86,5 @@
         	<origin rpy  = "0 -0 0" xyz = "-0.32661 0.24108 -0.06"/>
         	<geometry>
-          		<mesh scale=" 1 1 1" filename = "package://wheelchair_description_1/meshes/Right-Caster-Wheel_col.STL"/>
+          		<mesh scale=" 1 1 1" filename = "package://wheelchair_1_description/meshes/Right-Caster-Wheel_col.STL"/>
         	</geometry>
       	</collision>
@@ -98,5 +98,5 @@
 		  	<origin rpy = "0 -0 0" xyz = "-0.35956 0.24291 -0.1517"/>
 		  	<geometry>
-		  		<mesh scale=" 1 1 1" filename = "package://wheelchair_description_1/meshes/Right-Caster-Yaw.STL"/>
+		  		<mesh scale=" 1 1 1" filename = "package://wheelchair_1_description/meshes/Right-Caster-Yaw.STL"/>
 		  	</geometry>
 		</visual>
@@ -104,5 +104,5 @@
         	<origin rpy = "0 -0 0" xyz = "-0.35956 0.24291 -0.1517"/>
         	<geometry>
-          		<mesh scale=" 1 1 1" filename = "package://wheelchair_description_1/meshes/Right-Caster-Yaw_col.STL"/>
+          		<mesh scale=" 1 1 1" filename = "package://wheelchair_1_description/meshes/Right-Caster-Yaw_col.STL"/>
         	</geometry>
      	</collision>
@@ -116,5 +116,5 @@
 	  		<origin rpy  = "0 -0 0" xyz = "0 0.26808 -0.305"/>
 	  		<geometry>
-		  		<mesh scale=" 1 1 1" filename = "package://wheelchair_description_1/meshes/Right-Wheel.STL"/>
+		  		<mesh scale=" 1 1 1" filename = "package://wheelchair_1_description/meshes/Right-Wheel.STL"/>
 		  	</geometry>
 	  	</visual>
@@ -122,5 +122,5 @@
         	<origin rpy  = "0 -0 0" xyz = "0 0.26808 -0.305"/>
         	<geometry>
-          		<mesh scale=" 1 1 1" filename = "package://wheelchair_description_1/meshes/Right-Wheel_col.STL"/>
+          		<mesh scale=" 1 1 1" filename = "package://wheelchair_1_description/meshes/Right-Wheel_col.STL"/>
         	</geometry>
       	</collision>
@@ -178,6 +178,6 @@
      	</actuator>
       	<joint name="Wheelchair_base_Left_Wheel">
-        	<hardwareInterface>hardware_interface/VelocityJointInterface</hardwareInterface>
-        	<!-- <hardwareInterface>hardware_interface/EffortJointInterface</hardwareInterface> -->
+        	<Interface>hardware_interface/VelocityJointInterface</Interface>
+        	<!-- <Interface>hardware_interface/EffortJointInterface</Interface> -->
       	</joint>
     </transmission>
@@ -188,6 +188,6 @@
       	</actuator>
       	<joint name="Wheelchair_base_Right_Wheel">
-        	<hardwareInterface>hardware_interface/VelocityJointInterface</hardwareInterface>
-        	<!-- <hardwareInterface>hardware_interface/EffortJointInterface</hardwareInterface> -->
+        	<Interface>hardware_interface/VelocityJointInterface</Interface>
+        	<!-- <Interface>hardware_interface/EffortJointInterface</Interface> -->
       	</joint>
     </transmission>

File: Wheelchair_1/wheelchair_description_1/urdf/wheelchair.urdf (robot description, URDF)
Before this commit: robot wheelchair, 7 links, 6 joints
Links:
- link base_link: mass 4.78178 -> 54.78178
Joints:
- removed joint Wheelchair-base-Left-Wheel
- removed joint Wheelchair-base-Right-Wheel
- added joint Wheelchair_base_Left_Wheel: type revolute, parent base_link, child Left-Wheel, origin xyz=-0 0.26808 0.305, axis 0 1 0, limit lower=-1000 upper=1000 effort=100 velocity=10
- added joint Wheelchair_base_Right_Wheel: type revolute, parent base_link, child Right-Wheel, origin xyz=0 -0.26808 0.305, axis 0 1 0, limit lower=-1000 upper=1000 effort=100 velocity=10

File: Wheelchair_2/wheelchair_description/urdf/wheelchair.urdf.xacro (robot description, xacro)
@@ -380,9 +380,9 @@
     <type>transmission_interface/SimpleTransmission</type>
     <actuator name="SwingL_motor">
-      <hardwareInterface>PositionJointInterface</hardwareInterface>
+      <Interface>PositionJointInterface</Interface>
       <mechanicalReduction>1</mechanicalReduction>
     </actuator>
     <joint name="SwingL_rev">
-      <hardwareInterface>hardware_interface/EffortJointInterface</hardwareInterface>
+      <Interface>hardware_interface/EffortJointInterface</Interface>
     </joint>
   </transmission>
@@ -390,9 +390,9 @@
     <type>transmission_interface/SimpleTransmission</type>
     <actuator name="SwingR_motor">
-      <hardwareInterface>PositionJointInterface</hardwareInterface>
+      <Interface>PositionJointInterface</Interface>
       <mechanicalReduction>1</mechanicalReduction>
     </actuator>
     <joint name="SwingR_rev">
-      <hardwareInterface>hardware_interface/EffortJointInterface</hardwareInterface>
+      <Interface>hardware_interface/EffortJointInterface</Interface>
     </joint>
   </transmission>
@@ -401,9 +401,9 @@
     <type>transmission_interface/SimpleTransmission</type>
     <actuator name="WheelL_motor">
-      <hardwareInterface>EffortJointInterface</hardwareInterface>
+      <!-- <Interface>EffortJointInterface</Interface> -->
       <mechanicalReduction>1</mechanicalReduction>
     </actuator>
     <joint name="WheelL_cont">
-      <hardwareInterface>hardware_interface/VelocityJointInterface</hardwareInterface>
+      <Interface>hardware_interface/VelocityJointInterface</Interface>
     </joint>
   </transmission>
@@ -411,9 +411,9 @@
     <type>transmission_interface/SimpleTransmission</type>
     <actuator name="WheelR_motor">
-      <hardwareInterface>EffortJointInterface</hardwareInterface>
+      <!-- <Interface>EffortJointInterface</Interface> -->
       <mechanicalReduction>1</mechanicalReduction>
     </actuator>
     <joint name="WheelR_cont">
-      <hardwareInterface>hardware_interface/VelocityJointInterface</hardwareInterface>
+      <Interface>hardware_interface/VelocityJointInterface</Interface>
     </joint>
   </transmission>
