Commit message: Uploading recordings and bag to csv script

File: Wheelchair_2/wheelchair_description/urdf/wheelchair_2.0.urdf.xacro (robot description, xacro)
@@ -11,8 +11,8 @@
     <inertial>
       <origin
-        xyz="-0.2 0 0.22652"
-        rpy="0 0 0" />
-      <mass
-        value="25.655" />
+        xyz="-0.21708 0 0.22652"
+        rpy="0 0 0" />
+      <mass
+        value="15.655" />
       <inertia
         ixx="0.18789"
@@ -299,4 +299,5 @@
       effort="0"
       velocity="10" />
+    <dynamics damping="1.0" friction="0.2"/>
   </joint>
   <joint name="WheelF_cont"  type="continuous">
@@ -313,4 +314,5 @@
       effort="0"
       velocity="10" />
+    <dynamics damping="1.0" friction="0.1"/>
   </joint>
   <joint  name="SwingR_rev" type="revolute">
@@ -344,4 +346,5 @@
       effort="43"
       velocity="16.25" />
+    <dynamics damping="1.0" friction="0.0"/>
   </joint>
   <joint name="SwingL_rev" type="revolute">
@@ -375,4 +378,5 @@
       effort="43"
       velocity="16.25" />
+    <dynamics damping="1.0" friction="0.0"/>
   </joint>
   <!-- add transmission to swing arm joints -->
