Commit message: remove caster damping

File: Wheelchair_1/wheelchair_1_description/urdf/wheelchair.urdf.xacro (robot description, xacro)
@@ -137,5 +137,5 @@
 	   <axis xyz="0 1 0"/>
 	   <limit effort= "10" lower = "${lower}" upper = "${upper}" velocity = "10"/>
-	   <dynamics damping = ".7" friction ="1.5"/>
+	   <!-- <dynamics damping = ".7" friction ="1.5"/> -->
 	</joint>
 	<joint name="Wheelchair-base-Left-Caster-Yaw" type="revolute">
@@ -145,5 +145,5 @@
 	   <axis xyz="0 0 -1"/>
 	   <limit effort= "100" lower = "${lower}" upper = "${upper}" velocity = "10"/>
-	   <dynamics damping = "0.7" friction ="1.5"/>
+	   <!-- <dynamics damping = "0.7" friction ="1.5"/> -->
 	</joint>
 	<joint name="Wheelchair_base_Left_Wheel" type="revolute">
@@ -153,5 +153,5 @@
 	   <axis xyz="0 1 0"/>
 	   <limit effort= "100" lower = "${lower}" upper = "${upper}" velocity = "10"/>
-	   <dynamics damping = "0" friction ="0"/>
+	   <!-- <dynamics damping = "0" friction ="0"/> -->
 	</joint>
 	<joint name="Right-Caster-Yaw-Right-Caster-Wheel" type="revolute">
@@ -168,5 +168,5 @@
 	   <axis xyz="0 0 1"/>
 	   <limit effort= "100" lower = "${lower}" upper = "${upper}" velocity = "10"/>
-	   <dynamics damping = "0.7" friction ="1.5"/>
+	   <!-- <dynamics damping = "0.7" friction ="1.5"/> -->
 	</joint>
 	<joint name="Wheelchair_base_Right_Wheel" type="revolute">
@@ -176,5 +176,5 @@
 	   <axis xyz="0 1 0"/>
 	   <limit effort= "100" lower = "${lower}" upper = "${upper}" velocity = "10"/>
-	   <dynamics damping = "0" friction ="0"/>
+	   <!-- <dynamics damping = "0" friction ="0"/> -->
 	</joint>
     <transmission name="Wheelchair_base_Left_Wheel-trans">

File: Wheelchair_2/wheelchair_description/urdf/wheelchair_2.0.urdf.xacro (robot description, xacro)
@@ -409,6 +409,6 @@
     </actuator>
     <joint name="WheelL_cont">
-      <!-- <hardwareInterface>hardware_interface/VelocityJointInterface</hardwareInterface> -->
-      <hardwareInterface>hardware_interface/EffortJointInterface</hardwareInterface>
+      <hardwareInterface>hardware_interface/VelocityJointInterface</hardwareInterface>
+      <!-- <hardwareInterface>hardware_interface/EffortJointInterface</hardwareInterface> -->
     </joint>
   </transmission>
@@ -420,6 +420,6 @@
     </actuator>
     <joint name="WheelR_cont">
-      <!-- <hardwareInterface>hardware_interface/VelocityJointInterface</hardwareInterface> -->
-      <hardwareInterface>hardware_interface/EffortJointInterface</hardwareInterface>
+      <hardwareInterface>hardware_interface/VelocityJointInterface</hardwareInterface>
+      <!-- <hardwareInterface>hardware_interface/EffortJointInterface</hardwareInterface> -->
     </joint>
   </transmission>
